File: Hardware/clock_board_revC/project/heron_clock.kicad_pcb (KiCad board)
At the start: 4 copper layers, 118 x 44 mm, 110 parts, among them J1 5V_IN, J10 PPS_B200_2, J2 PPS_IN, J3 REF_B210_1, J4 REF_B210_2, J5 REF_B200_1, J6 REF_B200_2, J7 PPS_B210_1, J8 PPS_B210_2, J9 PPS_B200_1, U1 LP5907MFX-3.3/NOPB, U2 TLV75533PDBVR, U3 SiT5155AI-FK-33E0-10.000000, U4 LMK1C1104PWR, U5 SN74LVC1G17DBVR, U6 SN74LVC125APWR

Commit message: update pcb silk screen and rack cad
Other:
- board text added: "+5V IN"
- board text added: "10 MHz + PPS to 4 SDRs"
- board text added: "5.5V MAX"
- board text added: "DNP - fit if needed"
- board text added: "Designed by Nathan Cohen for CU Boulder"
- board text added: "HERON Clock Distribution Board"
- board text added: "R23: 50 ohm PPS load"
- board text added: "Rev C - 10/2026"
- board text added: "U3 SiT5155: water-soluble flux only"
- board text removed: "+5V"
- board text removed: "HERON CLOCK DIST rev C SiT5155 10 MHz + PPS x4 water-soluble flux only"
