File: Hardware/clock_board_revC/project/heron_clock.kicad_pcb (KiCad board)
At the start: 4 copper layers, 118 x 44 mm, 110 parts, among them J1 5V_IN, J10 PPS_B200_2, J2 PPS_IN, J3 REF_B210_1, J4 REF_B210_2, J5 REF_B200_1, J6 REF_B200_2, J7 PPS_B210_1, J8 PPS_B210_2, J9 PPS_B200_1, U1 LP5907MFX-3.3/NOPB, U2 TLV75533PDBVR, U3 SiT5155AI-FK-33E0-10.000000, U4 LMK1C1104PWR, U5 SN74LVC1G17DBVR, U6 SN74LVC125APWR

Commit message: Change clock board rev C J1 to JST XH; add CadQuery uv env for the rack
The JST-GH power header SM02B-GHS-TB(LF)(SN) is out of stock at
Digi-Key. J1 is now a JST S2B-XH-A-1(LF)(SN): through-hole, side entry,
friction lock (D-040). The pinout does not change.

- power_conn.py swaps the footprint, places J1 between D2 and J8,
  routes +5 V to the old track, removes 3 GND stitch vias, and moves
  the J1, "+5V IN" and J8 "PPS" silk. make_revc.py calls it.
- New gerbers and fab outputs. DRC: 28 items, no new ones. ERC: 0.
  J1 is not in the CPL file now (through-hole).
- BOM, design.py, README, HARDWARE.md and DECISIONS.md updated.
- Rack models use the XH body. check_fit.py: 0 clashes, mate PASS.
- Hardware/payload_rack is now its own uv project with CadQuery 2.8.
  Run "uv run python check_fit.py" there. CLAUDE.md tells agents how.

Co-Authored-By: Claude Opus 5.5 <noreply@anthropic.com>
Parts:
- J1: footprint Connector_JST:JST_GH_SM02B-GHS-TB_1x02-1MP_P1.25mm_Horizontal -> Connector_JST:JST_XH_S2B-XH-A-1_1x02_P2.50mm_Horizontal
- moved J1 7.55 mm to (136.1, 107.8)
Routing:
- net Net-(J1-Pin_1): track 9.88 -> 17.2 mm
- net GND: track 376.2 -> 374.8 mm, vias 461 -> 458

Commit message: Add clock board rev D: jacks on the real SDR connectors, USB holes
Photos of a B210 and a B200 show the SDR rear edge order: GPS ANT,
10 MHz, USB-B, PPS, DC jack. The rev C jacks faced GPS ANT and 10 MHz,
so rev C must not be ordered (Q-015 b, D-042).

Rev D (Hardware/clock_board_revD):
- J3-J6 face the SDR 10 MHz SMA, J7-J10 face the PPS SMA.
- Board 118 x 60 mm (rack z 30 to 90). A 16 x 18 mm hole on each
  SDR USB-B axis (a notch at the right edge), with a 2 mm keep-out
  ring so the hole can grow without new layout. DC and GPS ANT stay
  free.
- New generator gen_pcb.py: footprints from the KiCad 10 library,
  hand routes for the filter columns, PPS chains and U3, Freerouting
  1.9.0 for the rest. DRC 0, unconnected 0, footprint errors 0,
  parity 0. ERC 0. No starved thermals, no KiCad 7 footprint notes.
- Same schematic and parts as rev C.

Also in this commit:
- Rev C: D2 gets the Panjit SOD-323HE land (D-041); README marks
  rev C as superseded.
- bom_sources.csv: Digi-Key part numbers from the team order.
- Rack model: 10 MHz/PPS SMA positions corrected, rev D board, USB
  openings in the rear plate. check_fit.py: 0 clashes, all 8 jacks
  0.000 mm. Fusion seed and parts follow.
- DECISIONS.md (D-041, D-042, Q-015), HARDWARE.md, CLAUDE.md.

Co-Authored-By: Claude Opus 5.5 <noreply@anthropic.com>
Parts:
- D2: footprint Diode_SMD:D_SOD-323F -> HERON_Clock:D_SOD-323HE_Panjit
Changed lines of the file:
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@@
 		(embedded_fonts no)
 	)
-	(footprint "Diode_SMD:D_SOD-323F"
-		(layer "F.Cu")
-		(at 132.65 113.375 180)
-		(descr "SOD-323F http://www.nxp.com/documents/outline_drawing/SOD323F.pdf")
-		(tags "SOD-323F")
-		(property "Reference" "D2"
-			(at -0.491756 -1.835259 0)
-			(layer "F.SilkS")
-			(effects
-				(font
-					(size 0.8 0.8)
-					(thickness 0.12)
-				)
-			)
-		)
-		(property "Value" "SS1030HEWS"
-			(at 0.1 1.9 180)
-			(layer "F.Fab")
-			(effects
-				(font
-					(size 1 1)
-					(thickness 0.15)
-				)
-			)
-		)
-		(property "Datasheet" ""
-			(at 0 0 180)
-			(layer "F.Fab")
-			(hide yes)
-			(effects
-				(font
-					(size 1.27 1.27)
-				)
-			)
-		)
-		(property "Description" ""
-			(at 0 0 180)
-			(layer "F.Fab")
-			(hide yes)
-			(effects
-				(font
-					(size 1.27 1.27)
-				)
-			)
-		)
-		(property "MPN" "SS1030HEWS_R1_00001"
-			(at 265.3 226.75 0)
-			(layer "F.Fab")
-			(hide yes)
-			(effects
-				(font
-					(size 1 1)
-					(thickness 0.15)
-				)
-			)
-		)
-		(property "Manufacturer" "Panjit"
-			(at 265.3 226.75 0)
-			(layer "F.Fab")
-			(hide yes)
-			(effects
-				(font
-					(size 1 1)
-					(thickness 0.15)
-				)
-			)
-		)
-		(attr smd)
-		(duplicate_pad_numbers_are_jumpers no)
-		(fp_line
-			(start -1.61 0.85)
-			(end 1.05 0.85)
-			(stroke
-				(width 0.12)
-				(type solid)
-			)
-			(layer "F.SilkS")
-		)
-		(fp_line
-			(start -1.61 -0.85)
-			(end 1.05 -0.85)
-			(stroke
-				(width 0.12)
-				(type solid)
-			)
-			(layer "F.SilkS")
-		)
-		(fp_line
-			(start -1.61 -0.85)
-			(end -1.61 0.85)
-			(stroke
-				(width 0.12)
-				(type solid)
-			)
-			(layer "F.SilkS")
-		)
-		(fp_line
-			(start 1.6 -0.95)
-			(end 1.6 0.95)
-			(stroke
-				(width 0.05)
-				(type solid)
-			)
-			(layer "F.CrtYd")
-		)
-		(fp_line
-			(start -1.6 0.95)
-			(end 1.6 0.95)
-			(stroke
-				(width 0.05)
-				(type solid)
-			)
-			(layer "F.CrtYd")
-		)
-		(fp_line
-			(start -1.6 -0.95)
-			(end 1.6 -0.95)
-			(stroke
-				(width 0.05)
-				(type solid)
-			)
-			(layer "F.CrtYd")
-		)
-		(fp_line
-			(start -1.6 -0.95)
-			(end -1.6 0.95)
-			(stroke
-				(width 0.05)
-				(type solid)
-			)
-			(layer "F.CrtYd")
-		)
-		(fp_line
-			(start 0.9 0.7)
-			(end -0.9 0.7)
-			(stroke
-				(width 0.1)
-				(type solid)
-			)
-			(layer "F.Fab")
-		)
-		(fp_line
-			(start 0.9 -0.7)
-			(end 0.9 0.7)
-			(stroke
-				(width 0.1)
-				(type solid)
-			)
-			(layer "F.Fab")
-		)
-		(fp_line
-			(start 0.2 0.35)
-			(end -0.3 0)
-			(stroke
-				(width 0.1)
-				(type solid)
-			)
-			(layer "F.Fab")
-		)
-		(fp_line
-			(start 0.2 0)
-			(end 0.45 0)
-			(stroke
-				(width 0.1)
-				(type solid)
-			)
-			(layer "F.Fab")
-		)
-		(fp_line
-			(start 0.2 -0.35)
-			(end 0.2 0.35)
-			(stroke
-				(width 0.1)
-				(type solid)
-			)
-			(layer "F.Fab")
-		)
-		(fp_line
-			(start -0.3 0)
-			(end 0.2 -0.35)
-			(stroke
-				(width 0.1)
-				(type solid)
-			)
-			(layer "F.Fab")
-		)
-		(fp_line
-			(start -0.3 0)
-			(end -0.5 0)
-			(stroke
-				(width 0.1)
-				(type solid)
-			)
-			(layer "F.Fab")
-		)
-		(fp_line
-			(start -0.3 -0.35)
-			(end -0.3 0.35)
-			(stroke
-				(width 0.1)
-				(type solid)
-			)
-			(layer "F.Fab")
-		)
-		(fp_line
-			(start -0.9 0.7)
-			(end -0.9 -0.7)
-			(stroke
-				(width 0.1)
-				(type solid)
-			)
-			(layer "F.Fab")
-		)
-		(fp_line
-			(start -0.9 -0.7)
-			(end 0.9 -0.7)
-			(stroke
-				(width 0.1)
-				(type solid)
-			)
-			(layer "F.Fab")
-		)
-		(fp_text user "${REFERENCE}"
-			(at 0 -1.85 180)
-			(layer "F.Fab")
-			(effects
-				(font
-					(size 1 1)
-					(thickness 0.15)
-				)
-			)
-		)
-		(pad "1" smd roundrect
-			(at -1.1 0 180)
-			(size 0.5 0.5)
-			(layers "F.Cu" "F.Mask" "F.Paste")
-			(roundrect_rratio 0.25)
-			(net "Net-(D2-K)")
-		)
-		(pad "2" smd roundrect
-			(at 1.1 0 180)
-			(size 0.5 0.5)
-			(layers "F.Cu" "F.Mask" "F.Paste")
-			(roundrect_rratio 0.25)
-			(net "Net-(D1-K)")
-		)
-		(embedded_fonts no)
-		(model "${KICAD10_3DMODEL_DIR}/Diode_SMD.3dshapes/D_SOD-323F.step"
-			(offset
-				(xyz 0 0 0)
-			)
-			(scale
-				(xyz 1 1 1)
-			)
-			(rotate
-				(xyz 0 0 0)
-			)
-		)
-	)
 	(footprint "Capacitor_SMD:C_0603_1608Metric"
 		(layer "F.Cu")
@@
 		)
 	)
+	(footprint "HERON_Clock:D_SOD-323HE_Panjit"
+		(layer "F.Cu")
+		(at 132.65 113.375 180)
+		(descr "SOD-323HE (Panjit). Large cathode pad under the body. Land from Panjit SS1030HEWS datasheet rev 06, page 3")
+		(tags "SOD-323HE diode Panjit")
+		(property "Reference" "D2"
+			(at -0.95 -1.645448 0)
+			(layer "F.SilkS")
+			(effects
+				(font
+					(size 0.8 0.8)
+					(thickness 0.12)
+				)
+			)
+		)
+		(property "Value" "SS1030HEWS"
+			(at 0 1.6 180)
+			(layer "F.Fab")
+			(effects
+				(font
+					(size 0.8 0.8)
+					(thickness 0.12)
+				)
+			)
+		)
+		(property "Datasheet" ""
+			(at 0 0 180)
+			(layer "F.Fab")
+			(hide yes)
+			(effects
+				(font
+					(size 1.27 1.27)
+				)
+			)
+		)
+		(property "Description" ""
+			(at 0 0 180)
+			(layer "F.Fab")
+			(hide yes)
+			(effects
+				(font
+					(size 1.27 1.27)
+				)
+			)
+		)
+		(property "MPN" "SS1030HEWS_R1_00001"
+			(at 0 0 0)
+			(layer "F.Fab")
+			(hide yes)
+			(effects
+				(font
+					(size 1.27 1.27)
+					(thickness 0.15)
+				)
+			)
+		)
+		(property "Manufacturer" "Panjit"
+			(at 0 0 0)
+			(layer "F.Fab")
+			(hide yes)
+			(effects
+				(font
+					(size 1.27 1.27)
+					(thickness 0.15)
+				)
+			)
+		)
+		(attr smd)
+		(duplicate_pad_numbers_are_jumpers no)
+		(fp_line
+			(start -1.8 0.75)
+			(end 0 0.75)
+			(stroke
+				(width 0.12)
+				(type solid)
+			)
+			(layer "F.SilkS")
+		)
+		(fp_line
+			(start -1.8 -0.75)
+			(end 0 -0.75)
+			(stroke
+				(width 0.12)
+				(type solid)
+			)
+			(layer "F.SilkS")
+		)
+		(fp_line
+			(start -1.8 -0.75)
+			(end -1.8 0.75)
+			(stroke
+				(width 0.12)
+				(type solid)
+			)
+			(layer "F.SilkS")
+		)
+		(fp_rect
+			(start -1.85 -0.9)
+			(end 1.85 0.9)
+			(stroke
+				(width 0.05)
+				(type solid)
+			)
+			(fill no)
+			(layer "F.CrtYd")
+		)
+		(fp_line
+			(start -0.625 -0.65)
+			(end -0.625 0.65)
+			(stroke
+				(width 0.1)
+				(type solid)
+			)
+			(layer "F.Fab")
+		)
+		(fp_rect
+			(start -0.925 -0.65)
+			(end 0.925 0.65)
+			(stroke
+				(width 0.1)
+				(type solid)
+			)
+			(fill no)
+			(layer "F.Fab")
+		)
+		(fp_text user "${REFERENCE}"
+			(at 0 0 180)
+			(layer "F.Fab")
+			(effects
+				(font
+					(size 0.8 0.8)
+					(thickness 0.12)
+				)
+			)
+		)
+		(pad "1" smd roundrect
+			(at -0.675 0 180)
+			(size 1.85 1.1)
+			(layers "F.Cu" "F.Mask" "F.Paste")
+			(roundrect_rratio 0.1)
+			(net "Net-(D2-K)")
+		)
+		(pad "2" smd roundrect
+			(at 1.15 0 180)
+			(size 0.9 1)
+			(layers "F.Cu" "F.Mask" "F.Paste")
+			(roundrect_rratio 0.1)
+			(net "Net-(D1-K)")
+		)
+		(embedded_fonts no)
+	)
 	(footprint "Diode_SMD:D_SOD-523"
