File: Hardware/clock_board_revD/project/heron_clock.kicad_pcb (KiCad board)
At the start: 4 copper layers, 118 x 60 mm, 110 parts, among them J1 5V_IN, J10 PPS_B200_2, J2 PPS_IN, J3 REF_B210_1, J4 REF_B210_2, J5 REF_B200_1, J6 REF_B200_2, J7 PPS_B210_1, J8 PPS_B210_2, J9 PPS_B200_1, U1 LP5907MFX-3.3/NOPB, U2 TLV75533PDBVR, U3 SiT5155AI-FK-33E0-10.000000, U4 LMK1C1104PWR, U5 SN74LVC1G17DBVR, U6 SN74LVC125APWR

Commit message: Update clock board rev D: mid-edge holes, logo, 10 MHz ESD diodes
- Add mounting holes H5 and H6 at the middle of the long edges (D-043).
  The rack model gets the 2 matching rear-plate holes.
- Make the logo from the SVG. extract_logo.py reads the SVG and writes
  logo_polys.json. update_logo.py replaces only the logo polygons, so
  the copper does not change. The new SVG has one stray pixel less.
- Change the 10 MHz ESD diodes D4-D7 to the bidirectional TI
  TPD1E10B06DYAR (D-045). The AC-coupled 10 MHz goes below GND, and the
  unidirectional diode clipped it. The package and the layout do not
  change. Add the datasheet.
- Add mockup_dxf.py for the laser-cut fit mockup. The DXF and SVG
  outputs are not committed; run the script to make them.

Checks: DRC 0 violations, 0 unconnected, 0 parity issues; ERC 0.
Rack fit check: 0 clashes, all 8 jacks mate. Gerbers match the board.

Co-Authored-By: Claude Opus 5.5 <noreply@anthropic.com>
Parts:
- added H5: M3, MountingHole:MountingHole_3.2mm_M3_Pad_Via, F.Cu at (159.0, 104.0)
- added H6: M3, MountingHole:MountingHole_3.2mm_M3_Pad_Via, F.Cu at (159.0, 156.0)
- D4, D5, D6, D7: value TPD1E05U06 -> TPD1E10B06
- moved TP5 7.10 mm to (161.8, 147.6)
- moved C9 3.88 mm to (152.4, 154.2), turned to 180 degrees
- moved U6 2.00 mm to (160.0, 111.0)
- moved U3 0.30 mm to (156.5, 149.3)
Routing:
- net GND: track 400.4 -> 349.0 mm, vias 505 -> 472
- net /REF4_Y: track 58.7 -> 49.5 mm
- net /VIN_5V: track 60.7 -> 54.2 mm
- net /REF1_Y: track 57.1 -> 62.2 mm
- net /+3V3_CLK: track 130.9 -> 127.5 mm, vias 3 -> 4
- net /PPS_BUF: track 63.6 -> 60.5 mm
- net /PPS4_Y: track 54.8 -> 51.9 mm
- net /OSC_OE: track 5.71 -> 8.45 mm
- net /PPS1_Y: track 37.4 -> 39.0 mm
- net /REF2_Y: track 27.2 -> 28.6 mm
- net /+3V3_OSC: track 56.9 -> 55.9 mm
- net /PPS3_Y: track 23.4 -> 22.5 mm
- net Net-(J1-Pin_1): track 13.9 -> 13.1 mm
- net /PPS2_Y: track 4.93 -> 5.76 mm
